File: synth/eurorack-power-bus/eurorack-power-bus.kicad_pcb (KiCad board)
At the start: 2 copper layers, 100 x 90 mm, 22 parts, among them J1 IDC16, J10 IDC16, J11 IDC16, J12 IDC16, J13 IDC16, J14 IDC16, J15 IDC16, J16 IDC16, J17 IDC16, J18 IDC16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

Commit message: tracing
Routing:
- net Net-(J1-Pin_15): track 264.1 -> 304.7 mm
- net Net-(J1-Pin_13): track 264.9 -> 300.8 mm
- net Net-(J1-Pin_11): track 268.3 -> 298.7 mm
- net Net-(J1-Pin_7): track 264.6 -> 294.6 mm
- net Net-(J1-Pin_10): track 263.9 -> 289.9 mm
- net Net-(J1-Pin_5): track 264.0 -> 289.4 mm
- net Net-(J1-Pin_3): track 263.7 -> 284.9 mm
- net Net-(J1-Pin_1): track 265.9 -> 283.0 mm
