File: synth/mfos-wall-wart-eurorack-psu/mfos-wall-wart-eurorack-psu.kicad_pcb (KiCad board)
At the start: 2 copper layers, 80 x 100 mm, 70 parts, among them J1 JST5, J2 IDC16, K1 TestPoint_THTPad_D1.5mm_Drill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, K10 TestPoint_THTPad_D1.5mm_Drill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, K11 TestPoint_THTPad_D1.5mm_Drill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, K12 TestPoint_THTPad_D1.5mm_Drill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, K13 TestPoint_THTPad_D1.5mm_Drill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, K14 TestPoint_THTPad_D1.5mm_Drill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, K15 TestPoint_THTPad_D1.5mm_Drill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, K16 TestPoint_THTPad_D1.5mm_Drill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, K17 TestPoint_THTPad_D1.5mm_Drill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, K19 TestPoint_THTPad_D1.5mm_Drill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, K2 TestPoint_THTPad_D1.5mm_Drill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, K20 TestPoint_THTPad_D1.5mm_Drill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, K21 TestPoint_THTPad_D1.5mm_Drill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, K22 TestPoint_THTPad_D1.5mm_Drill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, K23 TestPoint_THTPad_D1.5mm_Drill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, K24 TestPoint_THTPad_D1.5mm_Drill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, K25 TestPoint_THTPad_D1.5mm_Drill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, K26 TestPoint_THTPad_D1.5mm_Drill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, K27 TestPoint_THTPad_D1.5mm_Drill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, K28 TestPoint_THTPad_D1.5mm_Drill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, K29 TestPoint_THTPad_D1.5mm_Drill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, K3 TestPoint_THTPad_D1.5mm_Drill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, K30 TestPoint_THTPad_D1.5mm_Drill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, K31 TestPoint_THTPad_D1.5mm_Drill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, K32 TestPoint_THTPad_D1.5mm_Drill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, K4 TestPoint_THTPad_D1.5mm_Drill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, K5 TestPoint_THTPad_D1.5mm_Drill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, K6 TestPoint_THTPad_D1.5mm_Drill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, K7 TestPoint_THTPad_D1.5mm_Drill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, K8 TestPoint_THTPad_D1.5mm_Drill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, K9 TestPoint_THTPad_D1.5mm_Drill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, M1 MountingHole_3.2mm_M3_DIN965_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, M2 MountingHole_3.2mm_M3_DIN965_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, M3 MountingHole_3.2mm_M3_DIN965_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, M4 MountingHole_3.2mm_M3_DIN965_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, U1 L7812CV, U2 L7805CV, U3 L7912CV

Commit message: add red stripe
Parts:
- added K1: TestPoint_THTPad_D1.5mm_Drill0.7mm, TestPoint:TestPoint_THTPad_D1.5mm_Drill0.7mm, F.Cu at (157.0, 144.2)
- added K10: TestPoint_THTPad_D1.5mm_Drill0.7mm, TestPoint:TestPoint_THTPad_D1.5mm_Drill0.7mm, F.Cu at (159.5, 146.7)
- added K11: TestPoint_THTPad_D1.5mm_Drill0.7mm, TestPoint:TestPoint_THTPad_D1.5mm_Drill0.7mm, F.Cu at (162.0, 146.7)
- added K12: TestPoint_THTPad_D1.5mm_Drill0.7mm, TestPoint:TestPoint_THTPad_D1.5mm_Drill0.7mm, F.Cu at (164.5, 146.7)
- added K13: TestPoint_THTPad_D1.5mm_Drill0.7mm, TestPoint:TestPoint_THTPad_D1.5mm_Drill0.7mm, F.Cu at (167.0, 146.7)
- added K14: TestPoint_THTPad_D1.5mm_Drill0.7mm, TestPoint:TestPoint_THTPad_D1.5mm_Drill0.7mm, F.Cu at (169.5, 146.7)
- added K15: TestPoint_THTPad_D1.5mm_Drill0.7mm, TestPoint:TestPoint_THTPad_D1.5mm_Drill0.7mm, F.Cu at (172.0, 146.7)
- added K16: TestPoint_THTPad_D1.5mm_Drill0.7mm, TestPoint:TestPoint_THTPad_D1.5mm_Drill0.7mm, F.Cu at (174.5, 146.7)
- added K2: TestPoint_THTPad_D1.5mm_Drill0.7mm, TestPoint:TestPoint_THTPad_D1.5mm_Drill0.7mm, F.Cu at (159.5, 144.2)
- added K3: TestPoint_THTPad_D1.5mm_Drill0.7mm, TestPoint:TestPoint_THTPad_D1.5mm_Drill0.7mm, F.Cu at (162.0, 144.2)
- added K4: TestPoint_THTPad_D1.5mm_Drill0.7mm, TestPoint:TestPoint_THTPad_D1.5mm_Drill0.7mm, F.Cu at (164.5, 144.2)
- added K5: TestPoint_THTPad_D1.5mm_Drill0.7mm, TestPoint:TestPoint_THTPad_D1.5mm_Drill0.7mm, F.Cu at (167.0, 144.2)
- added K6: TestPoint_THTPad_D1.5mm_Drill0.7mm, TestPoint:TestPoint_THTPad_D1.5mm_Drill0.7mm, F.Cu at (169.5, 144.2)
- added K7: TestPoint_THTPad_D1.5mm_Drill0.7mm, TestPoint:TestPoint_THTPad_D1.5mm_Drill0.7mm, F.Cu at (172.0, 144.2)
- added K8: TestPoint_THTPad_D1.5mm_Drill0.7mm, TestPoint:TestPoint_THTPad_D1.5mm_Drill0.7mm, F.Cu at (174.5, 144.2)
- added K9: TestPoint_THTPad_D1.5mm_Drill0.7mm, TestPoint:TestPoint_THTPad_D1.5mm_Drill0.7mm, F.Cu at (157.0, 146.7)

Commit message: rev 2
Parts:
- removed K1 (x2), K10 (x2), K11 (x2), K12 (x2), K13 (x2), K14 (x2), K15 (x2), K16 (x2), K17, K19, K2 (x2), K20, K21, K22, K23, K24, K25, K26, K27, K28, K29, K3 (x2), K30, K31, K32, K4 (x2), K5 (x2), K6 (x2), K7 (x2), K8 (x2), K9 (x2), REF**: TestPoint_THTPad_D1.5mm_Drill0.7mm, TestPoint:TestPoint_THTPad_D1.5mm_Drill0.7mm
- added D10: LED, LED_THT:LED_D3.0mm, F.Cu at (169.7, 140.6)
- added D11: LED, LED_THT:LED_D3.0mm, F.Cu at (169.7, 136.1)
- added D9: LED, LED_THT:LED_D3.0mm, F.Cu at (169.7, 145.1)
- added TP1: 12VAC, TestPoint:TestPoint_THTPad_D1.5mm_Drill0.7mm, F.Cu at (166.2, 52.5)
- added TP2: GND, TestPoint:TestPoint_THTPad_D1.5mm_Drill0.7mm, F.Cu at (166.2, 56.1)
- added TP3: +5V, TestPoint:TestPoint_THTPad_D1.5mm_Drill0.7mm, F.Cu at (151.2, 136.1)
- added TP4: +12V, TestPoint:TestPoint_THTPad_D1.5mm_Drill0.7mm, F.Cu at (151.2, 140.6)
- added TP5: -12V, TestPoint:TestPoint_THTPad_D1.5mm_Drill0.7mm, F.Cu at (151.2, 145.1)
- added TP6: GND, TestPoint:TestPoint_THTPad_D1.5mm_Drill0.7mm, F.Cu at (178.4, 136.0)
- moved R6 22.4 mm to (164.2, 145.1), turned to 180 degrees
- moved R5 22.2 mm to (164.2, 140.6), turned to 180 degrees
- moved R4 22.1 mm to (164.2, 136.1), turned to 180 degrees
- moved HS1 21.5 mm to (167.2, 122.6)
- moved HS2 21.5 mm to (141.2, 122.6)
- moved HS3 21.3 mm to (115.4, 122.4)
- moved J2 4.87 mm to (120.8, 138.6)
- moved D3 4.78 mm to (169.4, 101.2)
- moved C7 4.78 mm to (173.8, 101.4)
- moved C8 4.78 mm to (173.8, 104.9)
- moved D4 4.78 mm to (159.3, 105.2)
- moved C10 4.73 mm to (147.9, 107.5)
- moved C9 4.73 mm to (147.9, 98.8)
- moved D5 4.73 mm to (143.4, 101.1)
- moved D6 4.73 mm to (133.2, 105.1)
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Routing:
- net GND: track 279.9 -> 336.6 mm
- net Net-(D11-A): track 91.0 -> 114.1 mm
- net Net-(D1-K): track 32.5 -> 51.4 mm
- net Net-(D10-A): track 95.0 -> 112.9 mm
- net Net-(D9-A): track 99.8 -> 108.2 mm
- net Net-(D1-A): track 109.9 -> 105.5 mm
- net -12V: track 100.2 -> 98.2 mm
- net Net-(D2-K): track 138.0 -> 139.4 mm
- net +12V: track 108.9 -> 109.5 mm
Other:
- board text added: "12V"
- board text added: "@karczilla rev. 2 2024-07-21"
- board text added: "AC!"
- board text added: "MFOS Wall Wart Eurorack PSU"
- board text added: "optional"
- board text removed: "KLUDGE"
- board text removed: "MFOS Wall Wart Eurorack PSU @karczilla 2024-07-04"
