File: synth/mfos-wall-wart-eurorack-psu/mfos-wall-wart-eurorack-psu.kicad_pcb (KiCad board)
At the start: 2 copper layers, 80 x 100 mm, 47 parts, among them J1 JST5, J2 IDC16, M1 MountingHole_3.2mm_M3_DIN965_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, M2 MountingHole_3.2mm_M3_DIN965_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, M3 MountingHole_3.2mm_M3_DIN965_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, M4 MountingHole_3.2mm_M3_DIN965_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, U1 L7812CV, U2 L7805CV, U3 L7912CV

Commit message: ver2
Parts:
- moved TP2 3.55 mm to (169.7, 55.5)
- moved TP1 3.51 mm to (169.7, 52.8)
- moved D10 1.37 mm to (171.1, 140.6)
- moved D11 1.37 mm to (171.1, 136.1)
- moved D9 1.37 mm to (171.1, 145.1)
- moved R4 1.37 mm to (165.5, 136.1)
- moved R5 1.37 mm to (165.5, 140.6)
- moved R6 1.37 mm to (165.6, 145.1)
- moved TP3 1.37 mm to (152.6, 136.1)
- moved TP4 1.37 mm to (152.6, 140.6)
- moved TP5 1.37 mm to (152.6, 145.1)
Routing:
- net Net-(D11-A): track 114.1 -> 109.9 mm
- net Net-(D10-A): track 112.9 -> 108.8 mm
- net Net-(D1-K): track 51.4 -> 54.9 mm
- net GND: track 336.6 -> 333.3 mm
- net Net-(D2-K): track 139.4 -> 141.1 mm
Other:
- board text added: "- _/\/\_"
- board text added: "_/\/\_ +"
- board text added: "probing"
- board text removed: "12VAC"
