File: synth/mfos-wall-wart-eurorack-psu/mfos-wall-wart-eurorack-psu.kicad_sch (KiCad schematic)
At the start: 34 parts, among them J1 JST5, J2 IDC16, U1 L7812CV, U2 L7805CV, U3 L7912CV

Commit message: rev 2
Parts:
- added D10, D11, D9: LED, LED_THT:LED_D3.0mm, symbol Device:LED
- added TP1: 12VAC, TestPoint:TestPoint_THTPad_D1.5mm_Drill0.7mm, symbol Connector:TestPoint_Small
- added TP2, TP6: GND, TestPoint:TestPoint_THTPad_D1.5mm_Drill0.7mm, symbol Connector:TestPoint_Small
- added TP3: +5V, TestPoint:TestPoint_THTPad_D1.5mm_Drill0.7mm, symbol Connector:TestPoint_Small
- added TP4: +12V, TestPoint:TestPoint_THTPad_D1.5mm_Drill0.7mm, symbol Connector:TestPoint_Small
- added TP5: -12V, TestPoint:TestPoint_THTPad_D1.5mm_Drill0.7mm, symbol Connector:TestPoint_Small
- C1, C2, C3, C4, C5, C6: URL (none) -> https://www.taydaelectronics.com/3300uf-50v-105c-radial-ele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
- C10, C11, C12, C7, C8, C9: URL (none) -> https://www.taydaelectronics.com/1uf-50v-105c-radial-electr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
- D1, D2, D3, D4, D5, D6, D7, D8: URL (none) -> https://www.taydaelectronics.com/1n4004-diode-1a-400v.html
- HS1, HS2, HS3: URL (none) -> https://www.taydaelectronics.com/heatsink-to-220-4-fins-alu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
- J1: URL (none) -> https://www.taydaelectronics.com/5-pins-jst-xh-2-54-female-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
- R1, R2, R3: URL (none) -> https://www.taydaelectronics.com/10-x-resistor-2k-ohm-1-2w-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
- U1: URL (none) -> https://www.taydaelectronics.com/l7812cv-lm7812-l7812-volta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
- U2: URL (none) -> https://www.taydaelectronics.com/lm7805-l7805-7805-voltage-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
- U3: URL (none) -> https://www.taydaelectronics.com/l7912cv-lm7912-l7912-7912-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
Connections:
- net +12V: now also TP4.1
- net +5V: now also TP3.1
- net -12V: now also TP5.1
- net GND: now also D10.1 (K), D11.1 (K), D9.1 (K), TP2.1, TP6.1
- net at D1.1 (K), D2.2 (A), J1.1 (Pin_1): now also TP1.1
- net at J1.3 (Pin_3), R4.1: now also D11.2 (A)
- net at J1.4 (Pin_4), R5.1: now also D10.2 (A)
- net at J1.5 (Pin_5), R6.1: now also D9.2 (A)
Other:
- moved on the sheet: D4, D6, D8, J1, J2, R1, R2, R3, R4, R5, R6
