File: synth/mfos-wall-wart-eurorack-psu/mfos-wall-wart-eurorack-psu.kicad_sch (KiCad schematic)
At the start: 43 parts, among them J1 JST5, J2 IDC16, U1 L7812CV, U2 L7805CV, U3 L7912CV

Commit message: ver2
Other:
- note added: "(optional load resistors for probing)"
- note added: "(test points for probing)"
Changed lines of the file:
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@@
 	)
 	(junction
-		(at 60.96 54.61)
-		(diameter 0)
-		(color 0 0 0 0)
-	)
-	(junction
 		(at 99.06 74.93)
 		(diameter 0)
@@
 	)
 	(junction
+		(at 67.31 49.53)
+		(diameter 0)
+		(color 0 0 0 0)
+	)
+	(junction
 		(at 88.9 49.53)
 		(diameter 0)
@@
 	)
 	(junction
-		(at 64.77 62.23)
+		(at 231.14 64.77)
 		(diameter 0)
 		(color 0 0 0 0)
 	)
 	(junction
-		(at 231.14 64.77)
+		(at 67.31 62.23)
 		(diameter 0)
 		(color 0 0 0 0)
@@
 	(wire
 		(pts
-			(xy 64.77 57.15) (xy 64.77 62.23)
+			(xy 67.31 57.15) (xy 67.31 62.23)
 		)
 		(stroke
@@
 	(wire
 		(pts
-			(xy 60.96 49.53) (xy 88.9 49.53)
-		)
-		(stroke
-			(width 0)
-			(type default)
-		)
-	)
-	(wire
-		(pts
 			(xy 60.96 109.22) (xy 220.98 109.22)
 		)
@@
 	(wire
 		(pts
-			(xy 64.77 62.23) (xy 73.66 62.23)
-		)
-		(stroke
-			(width 0)
-			(type default)
-		)
-	)
-	(wire
-		(pts
 			(xy 187.96 71.12) (xy 187.96 72.39)
 		)
@@
 	(wire
 		(pts
-			(xy 55.88 62.23) (xy 64.77 62.23)
+			(xy 55.88 62.23) (xy 67.31 62.23)
 		)
 		(stroke
@@
 	(wire
 		(pts
-			(xy 60.96 54.61) (xy 60.96 59.69)
-		)
-		(stroke
-			(width 0)
-			(type default)
-		)
-	)
-	(wire
-		(pts
 			(xy 99.06 74.93) (xy 99.06 71.12)
 		)
@@
 	(wire
 		(pts
+			(xy 67.31 49.53) (xy 88.9 49.53)
+		)
+		(stroke
+			(width 0)
+			(type default)
+		)
+	)
+	(wire
+		(pts
 			(xy 198.12 81.28) (xy 204.47 81.28)
 		)
@@
 	(wire
 		(pts
+			(xy 67.31 49.53) (xy 67.31 54.61)
+		)
+		(stroke
+			(width 0)
+			(type default)
+		)
+	)
+	(wire
+		(pts
 			(xy 60.96 91.44) (xy 60.96 109.22)
 		)
@@
 	(wire
 		(pts
+			(xy 67.31 62.23) (xy 73.66 62.23)
+		)
+		(stroke
+			(width 0)
+			(type default)
+		)
+	)
+	(wire
+		(pts
 			(xy 187.96 35.56) (xy 187.96 34.29)
 		)
@@
 	(wire
 		(pts
-			(xy 60.96 49.53) (xy 60.96 54.61)
+			(xy 60.96 49.53) (xy 60.96 59.69)
 		)
 		(stroke
@@
 	(wire
 		(pts
-			(xy 60.96 54.61) (xy 64.77 54.61)
+			(xy 60.96 49.53) (xy 67.31 49.53)
 		)
 		(stroke
@@
 		)
 	)
+	(rectangle
+		(start 194.31 33.02)
+		(end 203.2 92.71)
+		(stroke
+			(width 0)
+			(type default)
+		)
+		(fill
+			(type none)
+		)
+	)
 	(text "+5V DC"
 		(exclude_from_sim no)
@@
 		)
 	)
+	(text "(optional load resistors for probing)"
+		(exclude_from_sim no)
+		(at 200.914 32.004 0)
+		(effects
+			(font
+				(size 1.27 1.27)
+			)
+		)
+	)
 	(text "CV"
 		(exclude_from_sim no)
@@
 		)
 	)
+	(text "(test points for probing)"
+		(exclude_from_sim no)
+		(at 252.984 88.9 0)
+		(effects
+			(font
+				(size 1.27 1.27)
+			)
+		)
+	)
 	(text "+5V LED"
 		(exclude_from_sim no)
@@
 		)
 	)
+	(text "(test points for probing)"
+		(exclude_from_sim no)
+		(at 74.676 52.578 0)
+		(effects
+			(font
+				(size 1.27 1.27)
+			)
+		)
+	)
 	(text "(to eurorack distribution bus...)"
 		(exclude_from_sim no)
@@
 	(symbol
 		(lib_id "Connector:TestPoint_Small")
-		(at 64.77 54.61 0)
+		(at 67.31 54.61 0)
 		(unit 1)
 		(exclude_from_sim no)
@@
 		(dnp no)
 		(property "Reference" "TP1"
-			(at 66.04 53.3399 0)
+			(at 68.58 53.3399 0)
 			(effects
 				(font
@@
 		)
 		(property "Value" "12VAC"
-			(at 65.278 54.61 0)
+			(at 67.818 54.61 0)
 			(effects
 				(font
@@
 		)
 		(property "Footprint" "TestPoint:TestPoint_THTPad_D1.5mm_Drill0.7mm"
-			(at 69.85 54.61 0)
+			(at 72.39 54.61 0)
 			(effects
 				(font
@@
 		)
 		(property "Datasheet" "~"
-			(at 69.85 54.61 0)
+			(at 72.39 54.61 0)
 			(effects
 				(font
@@
 		)
 		(property "Description" "Test Point"
-			(at 64.77 54.61 0)
+			(at 67.31 54.61 0)
 			(effects
 				(font
@@
 		)
 		(property "URL" ""
-			(at 64.77 54.61 0)
+			(at 67.31 54.61 0)
 			(effects
 				(font
@@
 	(symbol
 		(lib_id "Connector:TestPoint_Small")
-		(at 64.77 57.15 0)
+		(at 67.31 57.15 0)
 		(unit 1)
 		(exclude_from_sim no)
@@
 		(dnp no)
 		(property "Reference" "TP2"
-			(at 66.04 55.8799 0)
+			(at 68.58 55.8799 0)
 			(effects
 				(font
@@
 		)
 		(property "Value" "GND"
-			(at 65.278 57.15 0)
+			(at 67.818 57.15 0)
 			(effects
 				(font
@@
 		)
 		(property "Footprint" "TestPoint:TestPoint_THTPad_D1.5mm_Drill0.7mm"
-			(at 69.85 57.15 0)
+			(at 72.39 57.15 0)
 			(effects
 				(font
@@
 		)
 		(property "Datasheet" "~"
-			(at 69.85 57.15 0)
+			(at 72.39 57.15 0)
 			(effects
 				(font
@@
 		)
 		(property "Description" "Test Point"
-			(at 64.77 57.15 0)
+			(at 67.31 57.15 0)
 			(effects
 				(font
@@
 		)
 		(property "URL" ""
-			(at 64.77 57.15 0)
+			(at 67.31 57.15 0)
 			(effects
 				(font
