File: video/cvbs-decomposer/cvbs-decomposer.kicad_sch (KiCad schematic)
At the start: 29 parts, among them J1 CVBS_IN, J2 CVBS_THRU, J3 CSYNC_OUT, J4 VSYNC_OUT, J5 HSYNC_OUT, J6 FRAME_OUT, J8 ACTIVEVIDEO_OUT, J9 COLORBURST_OUT, U1 GS4981, U2 4013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

Commit message: fix 4538 terminations
Connections:
- net +5V: now also U5.11 (Clk-), U5.13 (R), U5.3 (R), U5.5 (Clk-)
- net GND: no longer U5.11 (Clk-), U5.13 (R), U5.3 (R), U5.5 (Clk-)

Commit message: rev 2
Parts:
- removed unit 4 of U3
- U3: value 4049 -> 4069/HC14
Connections:
- net at U1.5 (BACKP), U5.4 (Clk+): now also U3.9; no longer U3.11
- net at U4.5: now also U3.10; no longer U3.12
- net at J6.1 (Pin_1): now also U2.1 (Q)
Changed lines of the file:
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@@
 		)
 	)
-	(wire
-		(pts
-			(xy 199.39 85.09) (xy 214.63 85.09)
-		)
-		(stroke
-			(width 0)
-			(type default)
-		)
-	)
 	(polyline
 		(pts
@@
 	(wire
 		(pts
-			(xy 168.91 85.09) (xy 184.15 85.09)
+			(xy 168.91 85.09) (xy 214.63 85.09)
 		)
 		(stroke
@@
 	(rectangle
 		(start 55.88 123.19)
-		(end 167.64 163.83)
+		(end 207.01 163.83)
 		(stroke
 			(width 0)
@@
 			)
 		)
-		(property "Value" "4049"
+		(property "Value" "4069/HC14"
 			(at 191.77 52.832 0)
 			(effects
@@
 			)
 		)
-		(property "Value" "4049"
+		(property "Value" "4069/HC14"
 			(at 191.77 64.262 0)
 			(effects
@@
 			)
 		)
-		(property "Value" "4049"
+		(property "Value" "4069/HC14"
 			(at 191.77 41.402 0)
 			(effects
@@
 		(lib_id "4xxx:4049")
 		(at 191.77 102.87 0)
-		(unit 5)
+		(unit 4)
 		(exclude_from_sim no)
 		(in_bom yes)
@@
 			)
 		)
-		(property "Value" "4049"
+		(property "Value" "4069/HC14"
 			(at 191.77 98.552 0)
 			(effects
@@
 				(path "/60677854-96db-42b6-9827-28cf230d395c"
 					(reference "U3")
-					(unit 5)
+					(unit 4)
 				)
 			)
@@
 				)
 			)
-		)
-	)
-	(symbol
-		(lib_id "4xxx:4049")
-		(at 191.77 85.09 0)
-		(unit 4)
-		(exclude_from_sim no)
-		(in_bom yes)
-		(on_board yes)
-		(dnp no)
-		(property "Reference" "U3"
-			(at 191.77 78.232 0)
-			(effects
-				(font
-					(size 1.27 1.27)
-				)
-			)
-		)
-		(property "Value" "4049"
-			(at 191.77 80.772 0)
-			(effects
-				(font
-					(size 1.27 1.27)
-				)
-			)
-		)
-		(property "Footprint" ""
-			(at 191.77 85.09 0)
-			(effects
-				(font
-					(size 1.27 1.27)
-				)
-				(hide yes)
-			)
-		)
-		(property "Datasheet" "http://www.intersil.com/content/dam/intersil/documents/cd40/cd4049ubms.pdf"
-			(at 191.77 85.09 0)
-			(effects
-				(font
-					(size 1.27 1.27)
-				)
-				(hide yes)
-			)
-		)
-		(property "Description" "Hex Buffer Inverter"
-			(at 191.77 85.09 0)
-			(effects
-				(font
-					(size 1.27 1.27)
-				)
-				(hide yes)
-			)
-		)
-		(pin "2"
-		)
-		(pin "15"
-		)
-		(pin "6"
-		)
-		(pin "3"
-		)
-		(pin "11"
-		)
-		(pin "8"
-		)
-		(pin "12"
-		)
-		(pin "14"
-		)
-		(pin "7"
-		)
-		(pin "5"
-		)
-		(pin "1"
-		)
-		(pin "9"
-		)
-		(pin "10"
-		)
-		(pin "4"
-		)
-		(instances
-			(project "cvbs-decomposer"
-				(path "/60677854-96db-42b6-9827-28cf230d395c"
-					(reference "U3")
-					(unit 4)
-				)
-			)
