File: synth/mfos-wall-wart-eurorack-psu/kicad/mfos-wall-wart-eurorack-psu.kicad_pcb (KiCad board)
At the start: 2 copper layers, 80 x 100 mm, 47 parts, among them J1 JST5, J2 IDC16, M1 MountingHole_3.2mm_M3_DIN965_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, M2 MountingHole_3.2mm_M3_DIN965_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, M3 MountingHole_3.2mm_M3_DIN965_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, M4 MountingHole_3.2mm_M3_DIN965_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, U1 L7812CV, U2 L7805CV, U3 L7912CV

Commit message: rev2
Parts:
- J1: value JST5 -> JST-5
- J2: value IDC16 -> TERMINAL-4; footprint Connector_IDC:IDC-Header_2x08_P2.54mm_Vertical -> TerminalBlock_Phoenix:TerminalBlock_Phoenix_MKDS-1,5-4-5.08_1x04_P5.08mm_Horizontal
- TP5: value -12V -> GND
- TP6: value GND -> -12V
- moved TP6 30.9 mm to (147.5, 136.1)
- moved D10 1.88 mm to (172.9, 140.6)
- moved D11 1.88 mm to (172.9, 136.1)
- moved D9 1.88 mm to (172.9, 145.1)
- moved R4 1.88 mm to (167.4, 136.1)
- moved R5 1.88 mm to (167.4, 140.6)
- moved R6 1.88 mm to (167.5, 145.1)
- moved TP3 1.88 mm to (154.5, 136.1)
- moved TP4 1.88 mm to (154.5, 140.6)
- moved TP5 1.88 mm to (154.5, 145.1)
- moved J2 0.30 mm to (120.9, 138.9), turned to 0 degrees
Connections:
- J2 pad 2: -12V -> GND
- J2 pad 3: GND -> +12V
- J2 pad 4: GND -> +5V
- TP5 pad 1: -12V -> GND
- TP6 pad 1: GND -> -12V
Routing:
- net Net-(D9-A): track 108.3 -> 119.2 mm
- net Net-(D11-A): track 109.9 -> 118.4 mm
- net Net-(D10-A): track 108.8 -> 117.2 mm
- net -12V: track 98.2 -> 104.6 mm
- net +12V: track 109.5 -> 111.5 mm
- net Net-(D2-K): track 141.1 -> 139.1 mm
- net +5V: track 80.0 -> 78.2 mm
Other:
- board text removed: "CV"
- board text removed: "GATE"
