File: synth/mfos-wall-wart-eurorack-psu/kicad/mfos-wall-wart-eurorack-psu.kicad_pcb (KiCad board)
At the start: 2 copper layers, 80 x 100 mm, 47 parts, among them J1 JST-5, J2 TERMINAL-4, M1 MountingHole_3.2mm_M3_DIN965_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, M2 MountingHole_3.2mm_M3_DIN965_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, M3 MountingHole_3.2mm_M3_DIN965_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, M4 MountingHole_3.2mm_M3_DIN965_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, U1 L7812CV, U2 L7805CV, U3 L7912CV

Commit message: rev2
Parts:
- C10, C11, C12, C7, C8, C9: footprint Capacitor_THT:CP_Radial_Tantal_D5.0mm_P2.50mm -> Capacitor_THT:CP_Radial_D5.0mm_P2.50mm

Commit message: rev2
Parts:
- added C13: 100nF, Capacitor_THT:C_Disc_D3.0mm_W2.0mm_P2.50mm, F.Cu at (180.7, 104.4)
- added C14: 100nF, Capacitor_THT:C_Disc_D3.0mm_W2.0mm_P2.50mm, F.Cu at (154.6, 101.9)
- added C15: 100nF, Capacitor_THT:C_Disc_D3.0mm_W2.0mm_P2.50mm, F.Cu at (128.6, 104.4)
Routing:
- net GND: track 333.6 -> 362.3 mm
- net +5V: track 78.2 -> 87.3 mm
- net Net-(D9-A): track 119.2 -> 125.7 mm
- net +12V: track 111.5 -> 115.8 mm
- net Net-(D11-A): track 118.4 -> 114.4 mm, vias 0 -> 1
- net Net-(D10-A): track 117.2 -> 119.6 mm, vias 0 -> 1
- net Net-(D1-A): track 105.5 -> 104.7 mm
- net -12V: track 104.6 -> 105.3 mm
Other:
- board text added: "optional 'load' for probing"

Commit message: revisions
Parts:
- M1, M2, M3, M4: value MountingHole_3.2mm_M3_DIN965_Pad -> MountingHole_3.2mm_M3_Pad; footprint MountingHole:MountingHole_3.2mm_M3_DIN965_Pad -> MountingHole:MountingHole_3.2mm_M3_Pad
- R1, R2, R3: value 2K -> 2.4K
- R5, R6: value 500 -> 510
- renumbered D11 to L1, D10 to L2, D9 to L3

Commit message: fixes
Parts:
- C10, C11, C12, C7, C8, C9: footprint Capacitor_THT:CP_Radial_D5.0mm_P2.50mm -> Capacitor_THT:CP_Radial_Tantal_D5.0mm_P2.50mm
- moved C9 2.80 mm to (147.9, 101.7), turned to 90 degrees
- moved C14 2.72 mm to (154.9, 104.6), turned to 90 degrees
- moved C8 2.71 mm to (173.8, 107.7), turned to 90 degrees
- moved C11 2.21 mm to (122.2, 99.2), turned to -90 degrees
- moved D7 0.62 mm to (107.5, 101.7)
- moved D5 0.60 mm to (143.4, 101.7)
- moved D3 0.50 mm to (169.4, 101.7)
- moved C15 0.36 mm to (128.9, 104.6)
- moved C7 0.29 mm to (173.8, 101.7)
- moved C13 0.28 mm to (180.9, 104.6)
- moved C12 0.21 mm to (122.2, 105.2)
- moved D8 0.20 mm to (117.7, 105.2)
- moved C10 0.20 mm to (147.9, 107.7)
- moved D6 0.10 mm to (133.2, 105.2)
Routing:
- net -12V: track 105.3 -> 83.2 mm
- net GND: track 362.3 -> 377.3 mm
- net Net-(J1-Pin_5): track 125.7 -> 113.4 mm, vias 0 -> 1
- net +12V: track 115.8 -> 128.0 mm
- net Net-(J1-Pin_4): track 119.6 -> 111.8 mm
- net Net-(D1-A): track 104.7 -> 110.8 mm
- net Net-(D2-K): track 139.1 -> 143.7 mm
- net Net-(J1-Pin_3): track 114.4 -> 110.0 mm, vias 1 -> 3
- net +5V: track 87.3 -> 91.4 mm

Commit message: rev3
Parts:
- U1: value L7812CV -> L7805CV
- U2: value L7805CV -> L7812CV
- moved TP6 11.4 mm to (154.5, 145.1)
- moved R1 10.1 mm to (180.3, 112.2), turned to -90 degrees
- moved J1 8.05 mm to (125.1, 55.6), turned to 180 degrees
- moved TP5 7.33 mm to (147.2, 145.1)
- moved C15 2.50 mm to (128.9, 102.1), turned to -90 degrees
- moved U1 0.23 mm to (169.8, 111.0)
- moved U2 0.23 mm to (143.8, 111.0)
- moved U3 0.23 mm to (118.0, 111.0)
- moved HS1 0.20 mm to (167.2, 122.4)
- moved HS2 0.20 mm to (141.2, 122.4)
Connections:
- net Net-(J1-Pin_3) renamed +5V-LED
- net Net-(J1-Pin_4) renamed +12V-LED
- net Net-(J1-Pin_5) renamed -12V-LED
- C10 pad 1: +5V -> +12V
- C13 pad 1: +12V -> +5V
- C14 pad 1: +5V -> +12V
- C8 pad 1: +12V -> +5V
- D3 pad 2: +12V -> +5V
- D4 pad 1: +12V -> +5V
- D5 pad 2: +5V -> +12V
- D6 pad 1: +5V -> +12V
- R1 pad 1: +12V -> +5V
- R2 pad 1: +5V -> +12V
- U1 pad 3: +12V -> +5V
- U2 pad 3: +5V -> +12V
Routing:
- net GND: track 377.3 -> 515.0 mm
- net -12V: track 83.2 -> 115.6 mm
- net -12V-LED: track 113.4 -> 144.5 mm, vias 1 -> 0
- net Net-(D2-K): track 143.7 -> 173.8 mm, vias 0 -> 1
- net +5V: track 91.4 -> 117.8 mm
- net +12V-LED: track 111.8 -> 137.5 mm, vias 1 -> 0
- net +12V: track 128.0 -> 102.4 mm
- net +5V-LED: track 110.0 -> 132.2 mm, vias 3 -> 0
- net Net-(D1-A): track 110.8 -> 108.7 mm, vias 0 -> 1
Other:
- board text added: "@karczilla rev. 3 2024-07-30"
- board text added: "opt."
- board text removed: "@karczilla rev. 2 2024-07-21"
- board text removed: "optional 'load' for probing"

Commit message: prototyping board
Connections:
- net Net-(D1-K) renamed 12VAC
