File: synth/mfos-wall-wart-eurorack-psu/kicad/mfos-wall-wart-eurorack-psu.kicad_sch (KiCad schematic)
At the start: 43 parts, among them J1 JST5, J2 IDC16, U1 L7812CV, U2 L7805CV, U3 L7912CV

Commit message: rev2
Parts:
- removed J2: IDC16, Connector_IDC:IDC-Header_2x08_P2.54mm_Vertical, symbol Connector_Generic:Conn_02x08_Odd_Even
- added J2: TERMINAL-4, TerminalBlock_Phoenix:TerminalBlock_Phoenix_MKDS-1,5-4-5.08_1x04_P5.08mm_Horizontal, symbol Connector:Screw_Terminal_01x04
- J1: value JST5 -> JST-5
- R4, R5, R6: URL (none) -> ??
- TP5: value -12V -> GND
- TP6: value GND -> -12V
Connections:
- net +12V: now also J2.3 (Pin_3)
- net +5V: now also J2.4 (Pin_4)
- net -12V: now also TP6.1, J2.1 (Pin_1); no longer TP5.1
- net GND: now also TP5.1, J2.2 (Pin_2); no longer TP6.1
- no-connect marks 4 -> 0
Other:
- note added: "(probing)"
- note added: "(to bus)"
- note added: "(to front panel)"
- note removed: "(breakout connection to front panel)"
- note removed: "(test points for probing)"
- note removed: "(to eurorack distribution bus...)"
- note removed: "CV"
- note removed: "GATE"

Commit message: rev2
Parts:
- added C13, C14, C15: 100nF, Capacitor_THT:C_Disc_D3.0mm_W2.0mm_P2.50mm, symbol Device:C_Polarized_Small
- C10, C11, C12, C7, C8, C9: footprint Capacitor_THT:CP_Radial_Tantal_D5.0mm_P2.50mm -> Capacitor_THT:CP_Radial_D5.0mm_P2.50mm
- J2: URL ?? -> https://www.amazon.com/gp/product/B0CFYHDC7L/ref=ppx_yo_dt_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
- R1, R2, R3: value 2K -> 2.4K; URL https://www.taydaelectronics.com/10-x-resistor-2k-ohm-1-2w-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 -> https://www.taydaelectronics.com/resistors/1-4w-metal-film-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
- R4: URL ?? -> https://www.taydaelectronics.com/resistors/1-4w-metal-film-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
- R5, R6: value 500 -> 510; URL ?? -> https://www.taydaelectronics.com/resistors/1-4w-metal-film-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
Connections:
- net +12V: now also C13.1
- net +5V: now also C14.1
- net -12V: now also C15.2
- net GND: now also C13.2, C14.2, C15.1
Other:
- note removed: "(probing)"
- moved on the sheet: C1, C10, C11, C12, C2, C3, C4, C5, C6, C7, C8, C9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

Commit message: revisions
Parts:
- renumbered D11 to L1, D10 to L2, D9 to L3
Changed lines of the file:
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@@
 		(on_board yes)
 		(dnp no)
-		(property "Reference" "D10"
+		(property "Reference" "L2"
 			(at 45.466 111.252 0)
 			(effects
@@
 			(project "mfos-wall-wart-eurorack-psu"
 				(path "/173cde5c-ed8a-4b3f-9ce2-d2bc823d0323"
-					(reference "D10")
+					(reference "L2")
 					(unit 1)
 				)
@@
 		(on_board yes)
 		(dnp no)
-		(property "Reference" "D9"
+		(property "Reference" "L3"
 			(at 45.466 120.142 0)
 			(effects
@@
 			(project ""
 				(path "/173cde5c-ed8a-4b3f-9ce2-d2bc823d0323"
-					(reference "D9")
+					(reference "L3")
 					(unit 1)
 				)
@@
 		(on_board yes)
 		(dnp no)
-		(property "Reference" "D11"
+		(property "Reference" "L1"
 			(at 45.466 102.362 0)
 			(effects
@@
 			(project "mfos-wall-wart-eurorack-psu"
 				(path "/173cde5c-ed8a-4b3f-9ce2-d2bc823d0323"
-					(reference "D11")
+					(reference "L1")
 					(unit 1)
 				)

Commit message: fixes
Parts:
- C10, C11, C12, C7, C8, C9: footprint Capacitor_THT:CP_Radial_D5.0mm_P2.50mm -> Capacitor_THT:CP_Radial_Tantal_D5.0mm_P2.50mm; URL https://www.taydaelectronics.com/1uf-50v-105c-radial-electr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 -> https://www.taydaelectronics.com/1uf-35v-radial-tantalum-ca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
Other:
- moved on the sheet: C10, C12, C8

Commit message: rev3
Parts:
- removed U1: L7812CV, Package_TO_SOT_THT:TO-220-3_Vertical, symbol Regulator_Linear:L7812
- removed U2: L7805CV, Package_TO_SOT_THT:TO-220-3_Vertical, symbol Regulator_Linear:L7805
- added U1: L7805CV, Package_TO_SOT_THT:TO-220-3_Vertical, symbol Regulator_Linear:L7805
- added U2: L7812CV, Package_TO_SOT_THT:TO-220-3_Vertical, symbol Regulator_Linear:L7812
Connections:
- net +12V: now also C10.1, C14.1, D5.2 (A), D6.1 (K), R2.1, U2.3 (OUT); no longer C13.1, C8.1, D3.2 (A), D4.1 (K), R1.1
- net +5V: now also C13.1, C8.1, D3.2 (A), D4.1 (K), R1.1, U1.3 (OUT); no longer C10.1, C14.1, D5.2 (A), D6.1 (K), R2.1
- net GND: now also U1.2 (GND), U2.2 (GND)
- net at C1.1, C3.1, C5.1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: now also U1.1 (IN), U2.1 (IN)
Other:
- moved on the sheet: J2
