File: synth/eurorack-power-bus/kicad/eurorack-power-bus.kicad_pcb (KiCad board)
At the start: 2 copper layers, 245 x 50 mm, 37 parts, among them J1 IDC16, J10 IDC16, J11 IDC16, J12 IDC16, J13 IDC16, J14 IDC16, J15 IDC16, J16 IDC16, J17 IDC16, J18 IDC16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

Commit message: fixes
Parts:
- added M3: MountingHole_3.2mm_M3_Pad, MountingHole:MountingHole_3.2mm_M3_Pad, F.Cu at (151.9, 76.6)
- added M4: MountingHole_3.2mm_M3_Pad, MountingHole:MountingHole_3.2mm_M3_Pad, F.Cu at (151.9, 118.6)
- moved L3 18.7 mm to (142.7, 117.1)
- moved R3 18.7 mm to (127.2, 117.1)
- moved TP3 18.7 mm to (124.3, 117.1)
- moved TP{2 10.8 mm to (95.7, 117.1)
- moved L2 10.8 mm to (114.0, 117.1)
- moved R2 10.8 mm to (98.7, 117.1)
- moved TP4 2.21 mm to (58.7, 117.0)
- moved L1 1.82 mm to (85.5, 117.1)
- moved R1 1.82 mm to (70.1, 117.1)
- moved TP1 1.82 mm to (67.3, 117.1)
Routing:
- net GND: track 986.9 -> 967.6 mm
- net -12V: track 265.2 -> 258.7 mm
- net +5V: track 295.3 -> 290.9 mm
- net +12V: track 269.5 -> 267.8 mm

Commit message: fixes
Changed lines of the file:
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@@
 		)
 	)
-	(gr_text "Eurorack Power Bus\n(Passive)"
+	(gr_text "Eurorack Power Bus (Passive)"
 		(at 204.025 117.238375 0)
 		(layer "F.SilkS")
 		(effects
 			(font
-				(size 2 2)
+				(size 1 1)
 				(thickness 0.1)
 			)
