File: synth/synth-prototyping-pcb/kicad/synth-prototyping-pcb.kicad_pcb (KiCad board)
At the start: 2 copper layers, 53.3 x 100 mm, 31 parts, among them J1 Conn_02x16_Odd_Even, M1 MountingHole_3.2mm_M3_Pad

Commit message: prototyping board
Parts:
- removed the REF** at (125.4, 136.5)
- removed the REF** at (135.6, 136.5)
- removed the REF** at (150.8, 136.5)
- removed the REF** at (115.2, 136.5)
- removed the REF** at (133.0, 136.5)
- removed the REF** at (120.3, 136.5)
- removed the REF** at (148.3, 136.6)
- removed the REF** at (130.5, 136.5)
- removed the REF** at (143.2, 136.5)
- removed the REF** at (127.9, 136.5)
- removed the REF** at (110.2, 136.5)
- removed the REF** at (107.6, 136.5)
- removed the REF** at (122.9, 136.5)
- removed the REF** at (138.1, 136.5)
- removed the REF** at (117.8, 136.5)
- removed the REF** at (145.7, 136.5)
- removed the REF** at (105.1, 136.5)
- removed the REF** at (140.6, 136.5)
- removed the REF** at (112.7, 136.5)
- added REF**: Line, Connector_PinHeader_2.54mm:PinHeader_1x32_P2.54mm_Vertical, F.Cu at (103.4, 137.5)
- added REF**: Line, Connector_PinHeader_2.54mm:PinHeader_1x32_P2.54mm_Vertical, F.Cu at (131.3, 112.1)
- added REF**: Line, Connector_PinHeader_2.54mm:PinHeader_1x32_P2.54mm_Vertical, F.Cu at (128.8, 58.8)
- added REF**: Line, Connector_PinHeader_2.54mm:PinHeader_1x32_P2.54mm_Vertical, F.Cu at (108.4, 94.3)
- added REF**: Line, Connector_PinHeader_2.54mm:PinHeader_1x32_P2.54mm_Vertical, F.Cu at (108.4, 102.0)
- added REF**: Line, Connector_PinHeader_2.54mm:PinHeader_1x32_P2.54mm_Vertical, F.Cu at (131.3, 104.5)
- added REF**: Line, Connector_PinHeader_2.54mm:PinHeader_1x32_P2.54mm_Vertical, F.Cu at (108.4, 68.9)
- added REF**: Line, Connector_PinHeader_2.54mm:PinHeader_1x32_P2.54mm_Vertical, F.Cu at (138.9, 135.0)
- added REF**: Line, Connector_PinHeader_2.54mm:PinHeader_1x32_P2.54mm_Vertical, F.Cu at (131.3, 94.3)
- added REF**: Line, Connector_PinHeader_2.54mm:PinHeader_1x32_P2.54mm_Vertical, F.Cu at (108.4, 99.4)
- added REF**: Line, Connector_PinHeader_2.54mm:PinHeader_1x32_P2.54mm_Vertical, F.Cu at (108.4, 117.2)
- added REF**: Line, Connector_PinHeader_2.54mm:PinHeader_1x32_P2.54mm_Vertical, F.Cu at (131.3, 63.9)
- added REF**: Line, Connector_PinHeader_2.54mm:PinHeader_1x32_P2.54mm_Vertical, F.Cu at (108.4, 74.0)
- added REF**: Line, Connector_PinHeader_2.54mm:PinHeader_1x32_P2.54mm_Vertical, F.Cu at (108.4, 114.7)
- added REF**: Line, Connector_PinHeader_2.54mm:PinHeader_1x32_P2.54mm_Vertical, F.Cu at (131.3, 76.6)
- added REF**: Line, Connector_PinHeader_2.54mm:PinHeader_1x32_P2.54mm_Vertical, F.Cu at (131.3, 84.2)
- added REF**: Line, Connector_PinHeader_2.54mm:PinHeader_1x32_P2.54mm_Vertical, F.Cu at (108.4, 112.1)
- added REF**: Line, Connector_PinHeader_2.54mm:PinHeader_1x32_P2.54mm_Vertical, F.Cu at (108.4, 127.4)
- added REF**: Line, Connector_PinHeader_2.54mm:PinHeader_1x32_P2.54mm_Vertical, F.Cu at (131.3, 68.9)
- added REF**: Line, Connector_PinHeader_2.54mm:PinHeader_1x32_P2.54mm_Vertical, F.Cu at (108.4, 107.0)
- added REF**: Line, Connector_PinHeader_2.54mm:PinHeader_1x32_P2.54mm_Vertical, F.Cu at (131.3, 109.6)
- added REF**: Line, Connector_PinHeader_2.54mm:PinHeader_1x32_P2.54mm_Vertical, F.Cu at (108.4, 91.8)
- added REF**: Line, Connector_PinHeader_2.54mm:PinHeader_1x32_P2.54mm_Vertical, F.Cu at (108.4, 79.1)
- added REF**: Line, Connector_PinHeader_2.54mm:PinHeader_1x32_P2.54mm_Vertical, F.Cu at (131.3, 122.3)
- added REF**: Line, Connector_PinHeader_2.54mm:PinHeader_1x32_P2.54mm_Vertical, F.Cu at (108.4, 86.7)
- added REF**: Line, Connector_PinHeader_2.54mm:PinHeader_1x32_P2.54mm_Vertical, F.Cu at (108.4, 84.2)
- added REF**: Line, Connector_PinHeader_2.54mm:PinHeader_1x32_P2.54mm_Vertical, F.Cu at (108.4, 61.3)
- added REF**: Line, Connector_PinHeader_2.54mm:PinHeader_1x32_P2.54mm_Vertical, F.Cu at (131.3, 74.0)
- added REF**: Line, Connector_PinHeader_2.54mm:PinHeader_1x32_P2.54mm_Vertical, F.Cu at (131.3, 107.0)
- added REF**: Line, Connector_PinHeader_2.54mm:PinHeader_1x32_P2.54mm_Vertical, F.Cu at (111.0, 56.2)
- added REF**: Line, Connector_PinHeader_2.54mm:PinHeader_1x32_P2.54mm_Vertical, F.Cu at (131.3, 86.7)
- added REF**: Line, Connector_PinHeader_2.54mm:PinHeader_1x32_P2.54mm_Vertical, F.Cu at (108.4, 66.4)
- added REF**: Line, Connector_PinHeader_2.54mm:PinHeader_1x32_P2.54mm_Vertical, F.Cu at (131.3, 91.8)
- added REF**: Line, Connector_PinHeader_2.54mm:PinHeader_1x32_P2.54mm_Vertical, F.Cu at (131.3, 96.9)
- added REF**: Line, Connector_PinHeader_2.54mm:PinHeader_1x32_P2.54mm_Vertical, F.Cu at (131.3, 71.5)
- added REF**: Line, Connector_PinHeader_2.54mm:PinHeader_1x32_P2.54mm_Vertical, F.Cu at (131.3, 58.8)
- added REF**: Line, Connector_PinHeader_2.54mm:PinHeader_1x32_P2.54mm_Vertical, F.Cu at (108.4, 81.6)
- added REF**: Line, Connector_PinHeader_2.54mm:PinHeader_1x32_P2.54mm_Vertical, F.Cu at (151.6, 58.8)
- added REF**: Line, Connector_PinHeader_2.54mm:PinHeader_1x32_P2.54mm_Vertical, F.Cu at (149.1, 58.8)
- added REF**: Line, Connector_PinHeader_2.54mm:PinHeader_1x32_P2.54mm_Vertical, F.Cu at (103.4, 132.4)
- added REF**: Line, Connector_PinHeader_2.54mm:PinHeader_1x32_P2.54mm_Vertical, F.Cu at (131.3, 81.6)
- added REF**: Line, Connector_PinHeader_2.54mm:PinHeader_1x32_P2.54mm_Vertical, F.Cu at (103.4, 129.9)
- added REF**: Line, Connector_PinHeader_2.54mm:PinHeader_1x32_P2.54mm_Vertical, F.Cu at (108.4, 104.5)
- added REF**: Line, Connector_PinHeader_2.54mm:PinHeader_1x32_P2.54mm_Vertical, F.Cu at (131.3, 99.4)
- added REF**: Line, Connector_PinHeader_2.54mm:PinHeader_1x32_P2.54mm_Vertical, F.Cu at (131.3, 124.8)
- added REF**: Line, Connector_PinHeader_2.54mm:PinHeader_1x32_P2.54mm_Vertical, F.Cu at (103.3, 135.0)
- added REF**: Line, Connector_PinHeader_2.54mm:PinHeader_1x32_P2.54mm_Vertical, F.Cu at (108.4, 76.6)
- added REF**: Line, Connector_PinHeader_2.54mm:PinHeader_1x32_P2.54mm_Vertical, F.Cu at (131.3, 117.2)
- added REF**: Line, Connector_PinHeader_2.54mm:PinHeader_1x32_P2.54mm_Vertical, F.Cu at (138.9, 137.5)
- added REF**: Line, Connector_PinHeader_2.54mm:PinHeader_1x32_P2.54mm_Vertical, F.Cu at (131.3, 127.4)
- added REF**: Line, Connector_PinHeader_2.54mm:PinHeader_1x32_P2.54mm_Vertical, F.Cu at (111.0, 51.2)
- added REF**: Line, Connector_PinHeader_2.54mm:PinHeader_1x32_P2.54mm_Vertical, F.Cu at (108.4, 58.8)
- added REF**: Line, Connector_PinHeader_2.54mm:PinHeader_1x32_P2.54mm_Vertical, F.Cu at (108.4, 71.5)
- added REF**: Line, Connector_PinHeader_2.54mm:PinHeader_1x32_P2.54mm_Vertical, F.Cu at (131.3, 79.1)
- added REF**: Line, Connector_PinHeader_2.54mm:PinHeader_1x32_P2.54mm_Vertical, F.Cu at (111.0, 53.7)
- added REF**: Line, Connector_PinHeader_2.54mm:PinHeader_1x32_P2.54mm_Vertical, F.Cu at (108.4, 63.9)
- added REF**: Line, Connector_PinHeader_2.54mm:PinHeader_1x32_P2.54mm_Vertical, F.Cu at (131.3, 66.4)
- added REF**: Line, Connector_PinHeader_2.54mm:PinHeader_1x32_P2.54mm_Vertical, F.Cu at (108.4, 96.9)
- added REF**: Line, Connector_PinHeader_2.54mm:PinHeader_1x32_P2.54mm_Vertical, F.Cu at (131.3, 119.7)
- added REF**: Line, Connector_PinHeader_2.54mm:PinHeader_1x32_P2.54mm_Vertical, F.Cu at (126.2, 58.8)
- added REF**: Line, Connector_PinHeader_2.54mm:PinHeader_1x32_P2.54mm_Vertical, F.Cu at (108.4, 89.3)
- added REF**: Line, Connector_PinHeader_2.54mm:PinHeader_1x32_P2.54mm_Vertical, F.Cu at (131.3, 114.7)
- added REF**: Line, Connector_PinHeader_2.54mm:PinHeader_1x32_P2.54mm_Vertical, F.Cu at (108.4, 124.8)
- added REF**: Line, Connector_PinHeader_2.54mm:PinHeader_1x32_P2.54mm_Vertical, F.Cu at (131.3, 102.0)
- added REF**: Line, Connector_PinHeader_2.54mm:PinHeader_1x32_P2.54mm_Vertical, F.Cu at (131.3, 61.3)
- added REF**: Line, Connector_PinHeader_2.54mm:PinHeader_1x32_P2.54mm_Vertical, F.Cu at (108.4, 119.7)
- added REF**: Line, Connector_PinHeader_2.54mm:PinHeader_1x32_P2.54mm_Vertical, F.Cu at (108.4, 109.6)
- added REF**: Line, Connector_PinHeader_2.54mm:PinHeader_1x32_P2.54mm_Vertical, F.Cu at (105.9, 58.8)
- added REF**: Line, Connector_PinHeader_2.54mm:PinHeader_1x32_P2.54mm_Vertical, F.Cu at (131.3, 89.3)
- added REF**: Line, Connector_PinHeader_2.54mm:PinHeader_1x32_P2.54mm_Vertical, F.Cu at (108.4, 122.3)
- M1 (x4): value MountingHole_3.2mm_M3_Pad -> MountingHole_3.2mm_M3_DIN965_Pad; footprint MountingHole:MountingHole_3.2mm_M3_Pad -> MountingHole:MountingHole_3.2mm_M3_DIN965_Pad
- REF**: value PinHeader_1x32_P2.54mm_Vertical -> Line
- TP1: value TestPoint_Small -> +5V; footprint TestPoint:TestPoint_Plated_Hole_D2.0mm -> TestPoint:TestPoint_THTPad_2.0x2.0mm_Drill1.0mm
- TP2: value TestPoint_Small -> GND; footprint TestPoint:TestPoint_Plated_Hole_D2.0mm -> TestPoint:TestPoint_THTPad_2.0x2.0mm_Drill1.0mm
- TP3: value TestPoint_Small -> +12V; footprint TestPoint:TestPoint_Plated_Hole_D2.0mm -> TestPoint:TestPoint_THTPad_2.0x2.0mm_Drill1.0mm
- TP4: value TestPoint_Small -> -12V; footprint TestPoint:TestPoint_THTPad_1.5x1.5mm_Drill0.7mm -> TestPoint:TestPoint_THTPad_2.0x2.0mm_Drill1.0mm
- TP5: value TestPoint_Small -> CV; footprint TestPoint:TestPoint_Plated_Hole_D2.0mm -> TestPoint:TestPoint_THTPad_2.0x2.0mm_Drill1.0mm
- TP6: value TestPoint_Small -> GATE; footprint TestPoint:TestPoint_Plated_Hole_D2.0mm -> TestPoint:TestPoint_THTPad_2.0x2.0mm_Drill1.0mm
- moved TP5 97.0 mm to (132.4, 135.6)
- moved TP6 92.3 mm to (135.7, 135.6)
- moved TP4 83.2 mm to (119.2, 135.6)
- moved TP2 83.1 mm to (122.5, 135.6)
- moved TP3 83.1 mm to (125.8, 135.6)
- moved TP1 83.0 mm to (129.1, 135.6)
- moved REF** 77.7 mm to (103.4, 58.8), turned to 0 degrees
- moved M1 1.92 mm to (151.5, 145.7)
- moved M1 1.92 mm to (151.5, 52.7)
- moved J1 0.85 mm to (118.6, 145.2)
- moved M1 0.35 mm to (103.5, 145.7)
- moved M1 0.35 mm to (103.5, 52.7)
Connections:
- J1 pad 13: unconnected-(J1-Pin_13-Pad13) -> CV
- J1 pad 15: unconnected-(J1-Pin_15-Pad15) -> GATE
Routing:
- net (no net): track 152.4 -> 1496.1 mm
- net line: track 1270.0 -> 0.00 mm
- net GND: track 0.00 -> 25.3 mm
- net +12V: track 0.00 -> 10.8 mm
- net -12V: track 0.00 -> 10.8 mm
- net +5V: track 0.00 -> 10.5 mm
- net CV: track 0.00 -> 10.2 mm
- net GATE: track 0.00 -> 9.89 mm
Other:
- board size 53.3 x 100 mm -> 55 x 100 mm
- board text added: "MESSIËR"
